File: extras/auto_band_pass_filter.sch (EAGLE design)
At the start: 37 parts, among them M1 ARDUINO-PRO-MINI-3.3V, U1 FAIRCHILD_FST3253MXFAIRCHILD_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, U2 FAIRCHILD_FST3253MXFAIRCHILD_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

Commit message: ABPF
Parts:
- removed CZ12: 100nF, capacitor-wima:C2,5-3
- added C15, C16: 100nF, capacitor-wima:C2,5-3
Connections:
- net GND: now also C15.2, C16.2; no longer CZ12.1
- net VCC: now also C15.1, C16.1; no longer CZ12.2
Changed lines of the file:
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@@
 <part name="GND9" library="SparkFun-PowerSymbols" library_urn="urn:adsk.eagle:library:530" deviceset="GND" device=""/>
 <part name="GND10" library="SparkFun-PowerSymbols" library_urn="urn:adsk.eagle:library:530" deviceset="GND" device=""/>
-<part name="CZ12" library="capacitor-wima" library_urn="urn:adsk.eagle:library:116" deviceset="C" device="2,5-3" package3d_urn="urn:adsk.eagle:package:5436/1" value="100nF"/>
-<part name="GND12" library="SparkFun-PowerSymbols" library_urn="urn:adsk.eagle:library:530" deviceset="GND" device=""/>
+<part name="C15" library="capacitor-wima" library_urn="urn:adsk.eagle:library:116" deviceset="C" device="2,5-3" package3d_urn="urn:adsk.eagle:package:5436/1" value="100nF"/>
 <part name="L8" library="ngspice-simulation" library_urn="urn:adsk.eagle:library:527439" deviceset="L" device="" value="0.27uH"/>
 <part name="L4" library="ngspice-simulation" library_urn="urn:adsk.eagle:library:527439" deviceset="L" device="" value="2uH"/>
@@
 <part name="R8" library="Resistor" library_urn="urn:adsk.eagle:library:16378527" deviceset="R-US" device="AXIAL-7.2MM-PITCH" package3d_urn="urn:adsk.eagle:package:16378561/2" technology="_" value="75"/>
 <part name="GND3" library="SparkFun-PowerSymbols" library_urn="urn:adsk.eagle:library:530" deviceset="GND" device=""/>
+<part name="C16" library="capacitor-wima" library_urn="urn:adsk.eagle:library:116" deviceset="C" device="2,5-3" package3d_urn="urn:adsk.eagle:package:5436/1" value="100nF"/>
 </parts>
 <sheets>
@@
 <attribute name="VALUE" x="-127" y="162.306" size="1.778" layer="96" align="top-center"/>
 </instance>
-<instance part="CZ12" gate="G$1" x="-58.42" y="200.66" smashed="yes" rot="R180">
-<attribute name="NAME" x="-54.864" y="200.279" size="1.778" layer="95"/>
-<attribute name="VALUE" x="-54.864" y="205.359" size="1.778" layer="96"/>
-</instance>
-<instance part="GND12" gate="1" x="-58.42" y="193.04" smashed="yes">
-<attribute name="VALUE" x="-58.42" y="190.246" size="1.778" layer="96" align="top-center"/>
+<instance part="C15" gate="G$1" x="-53.34" y="210.82" smashed="yes" rot="R180">
+<attribute name="NAME" x="-49.784" y="210.439" size="1.778" layer="95"/>
+<attribute name="VALUE" x="-49.784" y="215.519" size="1.778" layer="96"/>
 </instance>
 <instance part="L8" gate="G$1" x="-165.1" y="203.2" smashed="yes" rot="R90">
@@
 <instance part="GND3" gate="1" x="-177.8" y="228.6" smashed="yes" rot="R180">
 <attribute name="VALUE" x="-177.8" y="231.394" size="1.778" layer="96" rot="R180" align="top-center"/>
+</instance>
+<instance part="C16" gate="G$1" x="-281.94" y="210.82" smashed="yes" rot="R180">
+<attribute name="NAME" x="-278.384" y="210.439" size="1.778" layer="95"/>
+<attribute name="VALUE" x="-291.084" y="212.979" size="1.778" layer="96"/>
 </instance>
 </instances>
@@
 <wire x1="-264.16" y1="218.44" x2="-269.24" y2="218.44" width="0.1524" layer="91"/>
 <junction x="-269.24" y="218.44"/>
+<pinref part="C16" gate="G$1" pin="2"/>
+<wire x1="-281.94" y1="215.9" x2="-281.94" y2="218.44" width="0.1524" layer="91"/>
+<wire x1="-281.94" y1="218.44" x2="-269.24" y2="218.44" width="0.1524" layer="91"/>
 </segment>
 <segment>
@@
 <wire x1="-71.12" y1="218.44" x2="-71.12" y2="215.9" width="0.1524" layer="91"/>
 <junction x="-71.12" y="215.9"/>
+<pinref part="C15" gate="G$1" pin="2"/>
+<wire x1="-53.34" y1="215.9" x2="-68.58" y2="215.9" width="0.1524" layer="91"/>
+<junction x="-68.58" y="215.9"/>
 </segment>
 <segment>
@@
 <pinref part="GND10" gate="1" pin="GND"/>
 <wire x1="-167.64" y1="167.64" x2="-127" y2="167.64" width="0.1524" layer="91"/>
-</segment>
-<segment>
-<pinref part="CZ12" gate="G$1" pin="1"/>
-<pinref part="GND12" gate="1" pin="GND"/>
-<wire x1="-58.42" y1="198.12" x2="-58.42" y2="195.58" width="0.1524" layer="91"/>
 </segment>
 <segment>
@@
 <pinref part="SUPPLY2" gate="G$1" pin="VCC"/>
 <wire x1="-269.24" y1="195.58" x2="-264.16" y2="195.58" width="0.1524" layer="91"/>
+<pinref part="C16" gate="G$1" pin="1"/>
+<wire x1="-264.16" y1="208.28" x2="-281.94" y2="208.28" width="0.1524" layer="91"/>
+<junction x="-264.16" y="208.28"/>
 </segment>
 <segment>
@@
 <pinref part="SUPPLY3" gate="G$1" pin="VCC"/>
 <wire x1="-71.12" y1="205.74" x2="-71.12" y2="203.2" width="0.1524" layer="91"/>
-<pinref part="CZ12" gate="G$1" pin="2"/>
-<wire x1="-58.42" y1="205.74" x2="-73.66" y2="205.74" width="0.1524" layer="91"/>
-<junction x="-73.66" y="205.74"/>
-</segment>
-</net>
+<pinref part="C15" gate="G$1" pin="1"/>
+<wire x1="-53.34" y1="208.28" x2="-53.34" y2="205.74" width="0.1524" layer="91"/>
+<wire x1="-53.34" y1="205.74" x2="-71.12" y2="205.74" width="0.1524" layer="91"/>
+<junction x="-71.12" y="205.74"/>
+</segment>
+</net>

Commit message: ABPF
Connections:
- net GND: no longer C15.2
Changed lines of the file:
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@@
 <wire x1="-71.12" y1="218.44" x2="-71.12" y2="215.9" width="0.1524" layer="91"/>
 <junction x="-71.12" y="215.9"/>
-<pinref part="C15" gate="G$1" pin="2"/>
-<wire x1="-53.34" y1="215.9" x2="-68.58" y2="215.9" width="0.1524" layer="91"/>
-<junction x="-68.58" y="215.9"/>
 </segment>
 <segment>
